File: STM32/C80488/stmC80488/stmC80488.kicad_pcb (KiCad board)
At the start: 2 copper layers, 46 x 42.2 mm, 15 parts, among them J1 Conn_01x04_Pin, J10 Conn_01x12_Pin, J4 Conn_01x12_Pin, J5 Conn_01x01_Pin, J8 Conn_01x12_Pin, J9 Conn_01x12_Pin, SW1 TS-1101-C-W, U1 STM32F072C8Tx

Commit message: backup
Routing:
- net +3.3V: track 164.5 -> 167.7 mm
Changed lines of the file:
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@@
+	)
+	(segment
+		(start 148.325 78.55)
+		(end 150.215 76.66)
+		(width 0.3)
+		(layer "F.Cu")
+		(net 1)
 	)
 	(segment
@@
 	)
 	(segment
+		(start 150.215 76.66)
+		(end 152.6 76.66)
+		(width 0.3)
+		(layer "F.Cu")
+		(net 1)
+	)
+	(segment
 		(start 125.65 93.75)
 		(end 124.8 93.75)
@@
 	)
 	(segment
-		(start 145.275 81.6)
-		(end 146.0125 80.8625)
-		(width 0.3)
-		(layer "F.Cu")
-		(net 1)
-	)
-	(segment
 		(start 139.4 87.475)
-		(end 145.2875 81.5875)
+		(end 138.3625 87.475)
 		(width 0.3)
 		(layer "F.Cu")
@@
 	)
 	(segment
-		(start 145.3 81.575)
-		(end 145.275 81.575)
-		(width 0.3)
-		(layer "F.Cu")
-		(net 1)
-	)
-	(segment
-		(start 150.215 76.66)
-		(end 152.6 76.66)
-		(width 0.3)
-		(layer "F.Cu")
-		(net 1)
-	)
-	(segment
 		(start 120 95.025)
 		(end 121.375 96.4)
@@
 	)
 	(segment
-		(start 146.0125 80.8625)
-		(end 150.215 76.66)
-		(width 0.3)
-		(layer "F.Cu")
-		(net 1)
-	)
-	(segment
 		(start 116.8 76.46)
 		(end 116.8 74.3)
@@
 	)
 	(segment
-		(start 145.2875 81.5875)
-		(end 145.3 81.575)
-		(width 0.3)
-		(layer "F.Cu")
-		(net 1)
-	)
-	(segment
 		(start 116.8 74.3)
 		(end 118.3 72.8)
@@
 	)
 	(segment
+		(start 148.325 78.55)
+		(end 139.4 87.475)
+		(width 0.3)
+		(layer "F.Cu")
+		(net 1)
+	)
+	(segment
 		(start 148.14 104.915)
 		(end 148.14 108.4)
@@
 	)
 	(segment
-		(start 138.3625 87.475)
-		(end 139.4 87.475)
-		(width 0.3)
-		(layer "F.Cu")
-		(net 1)
-	)
-	(segment
 		(start 124.089999 83.749999)
 		(end 126.8 83.749999)
@@
 		(start 126.8 83.749999)
 		(end 126.8 84.4)
-		(width 0.3)
-		(layer "F.Cu")
-		(net 1)
-	)
-	(segment
-		(start 145.275 81.575)
-		(end 145.275 81.6)
 		(width 0.3)
 		(layer "F.Cu")
@@
 	)
 	(via
-		(at 146.0125 80.8625)
+		(at 148.325 78.55)
 		(size 1.5)
 		(drill 0.7)
@@
 		(width 0.3)
 		(layer "B.Cu")
+		(net 1)
+	)
+	(segment
+		(start 148.325 78.55)
+		(end 146.0125 80.8625)
+		(width 0.3)
+		(layer "B.Cu")
